File: mikser/Mikser_simulation/AmpConfig_Simulation/_autosave-AmpConfig_Simulation.kicad_sch (KiCad schematic)
At the start: 12 parts, among them U1 ${SIM.PARAMS}, U2 ${SIM.PARAMS}

Commit message: added amplification sumulation
Parts:
- R5: value ROR -> {ROR}
Changed lines of the file:
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@@
 			)
 		)
-		(property "Value" "ROR"
+		(property "Value" "{ROR}"
 			(at 203.2 46.99 90)
 			(effects
